File: BE_Amplificateur_Audio/BE_Amplificateur_Audio.sch (KiCad schematic (older format))
At the start: 50 parts, among them J2 Conn_01x02, J3 Conn_01x03, Q1 2N2907A, Q11 BD138, Q13 2N2222A, Q2 2N2907A, Q3 2N2907A, Q4 2N2222A, Q5 2N2222A, Q6 2N2907A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

Commit message: màj schematic + empreintes
Modification du schematic pour coller avec les instructions données.
Tentative de match des empreintes : à vérifier. Apparemment la lib d'empreinte donnée par le prof ne s'est pas chargée correctement : à vérfier !
Parts:
- removed ACHANGER (x2): TIP30C_Obsolete, digikey-footprints:TO-220-3, symbol dk_Transistors-Bipolar-BJT-Single:TIP30C_Obsolete
- removed ACHANGER: DIPxx-1Axx-12x, Relay_THT:Relay_StandexMeder_DIP_LowProfile, symbol Relay:DIPxx-1Axx-12x
- removed Achanger: BZX84Cxx, Diode_SMD:D_SOT-23_ANK, symbol Diode:BZX84Cxx
- removed Q1, Q2, Q3, Q6, Q7: 2N2907A, digikey-footprints:TO-18-3, symbol dk_Transistors-Bipolar-BJT-Single:2N2907A
- removed Q11: BD138, Package_TO_SOT_THT:TO-126-3_Vertical, symbol Transistor_BJT:BD138
- removed Q13, Q4, Q5: 2N2222A, digikey-footprints:TO-18-3, symbol dk_Transistors-Bipolar-BJT-Single:2N2222A
- added Dz1: BZX55C5V1, Be-Elec:D_DO-35_SOD27_P10.16mm_Horizontal, symbol Device:D_Zener_ALT
- added HS1, HS2: Heatsink, Heatsink:Heatsink_125x35x50mm_3xFixationM3, symbol Mechanical:Heatsink
- added Q1, Q2, Q3, Q6, Q7: 2N2907, Be-Elec:TO-18-3, symbol Device:Q_PNP_EBC
- added Q10: TIP32, Be-Elec:TO-126-3_Vertical, symbol Device:Q_PNP_BCE
- added Q11: BD138, Be-Elec:TO-126-3_Vertical, symbol Device:Q_PNP_ECB
- added Q12: TIP31, Be-Elec:TO-126-3_Vertical, symbol Device:Q_PNP_BCE
- added Q13, Q4, Q5: 2N2222, Package_TO_SOT_THT:TO-18-3, symbol Device:Q_NPN_EBC
- added U1: Relay_1CT, Relay_THT:Relay_StandexMeder_DIP_LowProfile, symbol BE_Amplificateur_Audio-cache:Relay:DIPxx-1Axx-12x
- C1, C2, C3, C4, C5, C6, C7, C8, C9: footprint (none) -> Be-Elec:CP_Radial_D12.5mm_P5.00mm
- C10, C11: renamed from C?; footprint (none) -> Be-Elec:CP_Radial_D12.5mm_P5.00mm
- J2: footprint (none) -> Connector:JWT_A3963_1x02_P3.96mm_Vertical
- J3: footprint (none) -> Connector:FanPinHeader_1x03_P2.54mm_Vertical
- R1, R10, R11, R12, R13, R14, R15, R16, R17, R2, R3, R4, R5, R6, R7, R8, R9: footprint (none) -> Be-Elec:D_DO-35_SOD27_P10.16mm_Horizontal
- RV1, RV2: footprint (none) -> Be-Elec:Potentiometer_Bourns_3296W_Vertical
- U2: footprint (none) -> Connector_Audio:Jack_Horizontal
Connections:
- wire segments 143 -> 147

Commit message: màj empreintes
Empreintes màj. A verifier qd même pour voir si la lib du prof a bien marché.
A faire : empreinte du relai.
Parts:
- removed U1: Relay_1CT, Relay_THT:Relay_StandexMeder_DIP_LowProfile, symbol BE_Amplificateur_Audio-cache:Relay:DIPxx-1Axx-12x
- added U1: Relay_1CT, Relay_THT:Relay_StandexMeder_DIP_LowProfile, symbol Relay:DIPxx-1Axx-12x
- D1, D2: footprint Diode_THT:D_DO-35_SOD27_P7.62mm_Horizontal -> Be-Elec:D_DO-35_SOD27_P10.16mm_Horizontal
- HS1, HS2: footprint Heatsink:Heatsink_125x35x50mm_3xFixationM3 -> Be-Elec:Heatsink_Fischer_SK104-STC-STIC_35x13mm_2xDrill2.5mm
- J2: footprint Connector:JWT_A3963_1x02_P3.96mm_Vertical -> Be-Elec:PhoenixContact_MSTBVA_2,5_2-G-5,08_1x02_P5.08mm_Vertical
- J3: footprint Connector:FanPinHeader_1x03_P2.54mm_Vertical -> Be-Elec:PhoenixContact_MSTBVA_2,5_3-G-5,08_1x03_P5.08mm_Vertical
- Q13, Q4, Q5: footprint Package_TO_SOT_THT:TO-18-3 -> Be-Elec:TO-18-3
- Q8, Q9: footprint Package_TO_SOT_THT:TO-126-3_Vertical -> Be-Elec:TO-126-3_Vertical
- R1, R10, R11, R12, R13, R14, R15, R16, R17, R2, R3, R4, R5, R6, R7, R8, R9: footprint Be-Elec:D_DO-35_SOD27_P10.16mm_Horizontal -> Be-Elec:R_Axial_DIN0207_L6.3mm_D2.5mm_P10.16mm_Horizontal
- U2: footprint Connector_Audio:Jack_Horizontal -> Be-Elec:Jack_35RAPC2AV
Changed lines of the file:
@@
 F 0 "U2" H 1076 4417 50  0000 C CNN
 F 1 "Jack_Mono" H 1076 4326 50  0000 C CNN
-F 2 "Connector_Audio:Jack_Horizontal" H 1100 4350 50  0001 C CNN
+F 2 "Be-Elec:Jack_35RAPC2AV" H 1100 4350 50  0001 C CNN
 F 3 "" H 1100 4350 50  0001 C CNN
 	1    1050 4150
@@
 F 0 "R1" H 1720 4546 50  0000 L CNN
 F 1 "R" H 1720 4455 50  0000 L CNN
-F 2 "Be-Elec:D_DO-35_SOD27_P10.16mm_Horizontal" V 1580 4500 50  0001 C CNN
+F 2 "Be-Elec:R_Axial_DIN0207_L6.3mm_D2.5mm_P10.16mm_Horizontal" V 1580 4500 50  0001 C CNN
 F 3 "~" H 1650 4500 50  0001 C CNN
 	1    1650 4500
@@
 F 0 "R5" H 2170 3296 50  0000 L CNN
 F 1 "R" H 2170 3205 50  0000 L CNN
-F 2 "Be-Elec:D_DO-35_SOD27_P10.16mm_Horizontal" V 2030 3250 50  0001 C CNN
+F 2 "Be-Elec:R_Axial_DIN0207_L6.3mm_D2.5mm_P10.16mm_Horizontal" V 2030 3250 50  0001 C CNN
 F 3 "~" H 2100 3250 50  0001 C CNN
 	1    2100 3250
@@
 F 0 "R2" H 2270 4846 50  0000 L CNN
 F 1 "R" H 2270 4755 50  0000 L CNN
-F 2 "Be-Elec:D_DO-35_SOD27_P10.16mm_Horizontal" V 2130 4800 50  0001 C CNN
+F 2 "Be-Elec:R_Axial_DIN0207_L6.3mm_D2.5mm_P10.16mm_Horizontal" V 2130 4800 50  0001 C CNN
 F 3 "~" H 2200 4800 50  0001 C CNN
 	1    2200 4800
@@
 F 0 "R3" H 3070 4846 50  0000 L CNN
 F 1 "R" H 3070 4755 50  0000 L CNN
-F 2 "Be-Elec:D_DO-35_SOD27_P10.16mm_Horizontal" V 2930 4800 50  0001 C CNN
+F 2 "Be-Elec:R_Axial_DIN0207_L6.3mm_D2.5mm_P10.16mm_Horizontal" V 2930 4800 50  0001 C CNN
 F 3 "~" H 3000 4800 50  0001 C CNN
 	1    3000 4800
@@
 F 0 "R4" H 2670 2696 50  0000 L CNN
 F 1 "R" H 2670 2605 50  0000 L CNN
-F 2 "Be-Elec:D_DO-35_SOD27_P10.16mm_Horizontal" V 2530 2650 50  0001 C CNN
+F 2 "Be-Elec:R_Axial_DIN0207_L6.3mm_D2.5mm_P10.16mm_Horizontal" V 2530 2650 50  0001 C CNN
 F 3 "~" H 2600 2650 50  0001 C CNN
 	1    2600 2650
@@
 F 0 "R9" H 3420 2696 50  0000 L CNN
 F 1 "R" H 3420 2605 50  0000 L CNN
-F 2 "Be-Elec:D_DO-35_SOD27_P10.16mm_Horizontal" V 3280 2650 50  0001 C CNN
+F 2 "Be-Elec:R_Axial_DIN0207_L6.3mm_D2.5mm_P10.16mm_Horizontal" V 3280 2650 50  0001 C CNN
 F 3 "~" H 3350 2650 50  0001 C CNN
 	1    3350 2650
@@
 F 0 "R7" H 4420 2696 50  0000 L CNN
 F 1 "R" H 4420 2605 50  0000 L CNN
-F 2 "Be-Elec:D_DO-35_SOD27_P10.16mm_Horizontal" V 4280 2650 50  0001 C CNN
+F 2 "Be-Elec:R_Axial_DIN0207_L6.3mm_D2.5mm_P10.16mm_Horizontal" V 4280 2650 50  0001 C CNN
 F 3 "~" H 4350 2650 50  0001 C CNN
 	1    4350 2650
@@
 F 0 "R10" H 3420 3396 50  0000 L CNN
 F 1 "R" H 3420 3305 50  0000 L CNN
-F 2 "Be-Elec:D_DO-35_SOD27_P10.16mm_Horizontal" V 3280 3350 50  0001 C CNN
+F 2 "Be-Elec:R_Axial_DIN0207_L6.3mm_D2.5mm_P10.16mm_Horizontal" V 3280 3350 50  0001 C CNN
 F 3 "~" H 3350 3350 50  0001 C CNN
 	1    3350 3350
@@
 F 0 "R8" V 3943 3850 50  0000 C CNN
 F 1 "R" V 4034 3850 50  0000 C CNN
-F 2 "Be-Elec:D_DO-35_SOD27_P10.16mm_Horizontal" V 4080 3850 50  0001 C CNN
+F 2 "Be-Elec:R_Axial_DIN0207_L6.3mm_D2.5mm_P10.16mm_Horizontal" V 4080 3850 50  0001 C CNN
 F 3 "~" H 4150 3850 50  0001 C CNN
 	1    4150 3850
@@
 F 0 "R6" H 4420 5296 50  0000 L CNN
 F 1 "R" H 4420 5205 50  0000 L CNN
-F 2 "Be-Elec:D_DO-35_SOD27_P10.16mm_Horizontal" V 4280 5250 50  0001 C CNN
+F 2 "Be-Elec:R_Axial_DIN0207_L6.3mm_D2.5mm_P10.16mm_Horizontal" V 4280 5250 50  0001 C CNN
 F 3 "~" H 4350 5250 50  0001 C CNN
 	1    4350 5250
@@
 F 0 "R15" H 3420 6096 50  0000 L CNN
 F 1 "R" H 3420 6005 50  0000 L CNN
-F 2 "Be-Elec:D_DO-35_SOD27_P10.16mm_Horizontal" V 3280 6050 50  0001 C CNN
+F 2 "Be-Elec:R_Axial_DIN0207_L6.3mm_D2.5mm_P10.16mm_Horizontal" V 3280 6050 50  0001 C CNN
 F 3 "~" H 3350 6050 50  0001 C CNN
 	1    3350 6050
@@
 F 0 "R14" V 3693 5800 50  0000 C CNN
 F 1 "R" V 3784 5800 50  0000 C CNN
-F 2 "Be-Elec:D_DO-35_SOD27_P10.16mm_Horizontal" V 3830 5800 50  0001 C CNN
+F 2 "Be-Elec:R_Axial_DIN0207_L6.3mm_D2.5mm_P10.16mm_Horizontal" V 3830 5800 50  0001 C CNN
 F 3 "~" H 3900 5800 50  0001 C CNN
 	1    3900 5800
@@
 F 0 "Q9" H 5142 3296 50  0000 L CNN
 F 1 "BD139" H 5142 3205 50  0000 L CNN
-F 2 "Package_TO_SOT_THT:TO-126-3_Vertical" H 5150 3175 50  0001 L CIN
+F 2 "Be-Elec:TO-126-3_Vertical" H 5150 3175 50  0001 L CIN
 F 3 "http://www.st.com/internet/com/TECHNICAL_RESOURCES/TECHNICAL_LITERATURE/DATASHEET/CD00001225.pdf" H 4950 3250 50  0001 L CNN
 	1    4950 3250
@@
 F 0 "R11" H 5620 3796 50  0000 L CNN
 F 1 "R" H 5620 3705 50  0000 L CNN
-F 2 "Be-Elec:D_DO-35_SOD27_P10.16mm_Horizontal" V 5480 3750 50  0001 C CNN
+F 2 "Be-Elec:R_Axial_DIN0207_L6.3mm_D2.5mm_P10.16mm_Horizontal" V 5480 3750 50  0001 C CNN
 F 3 "~" H 5550 3750 50  0001 C CNN
 	1    5550 3750
@@
 F 0 "R12" H 5620 4246 50  0000 L CNN
 F 1 "R" H 5620 4155 50  0000 L CNN
-F 2 "Be-Elec:D_DO-35_SOD27_P10.16mm_Horizontal" V 5480 4200 50  0001 C CNN
+F 2 "Be-Elec:R_Axial_DIN0207_L6.3mm_D2.5mm_P10.16mm_Horizontal" V 5480 4200 50  0001 C CNN
 F 3 "~" H 5550 4200 50  0001 C CNN
 	1    5550 4200
@@
 F 0 "R13" H 6270 4246 50  0000 L CNN
 F 1 "R" H 6270 4155 50  0000 L CNN
-F 2 "Be-Elec:D_DO-35_SOD27_P10.16mm_Horizontal" V 6130 4200 50  0001 C CNN
+F 2 "Be-Elec:R_Axial_DIN0207_L6.3mm_D2.5mm_P10.16mm_Horizontal" V 6130 4200 50  0001 C CNN
 F 3 "~" H 6200 4200 50  0001 C CNN
 	1    6200 4200
@@
 F 0 "R17" H 8270 5346 50  0000 L CNN
 F 1 "R" H 8270 5255 50  0000 L CNN
-F 2 "Be-Elec:D_DO-35_SOD27_P10.16mm_Horizontal" V 8130 5300 50  0001 C CNN
+F 2 "Be-Elec:R_Axial_DIN0207_L6.3mm_D2.5mm_P10.16mm_Horizontal" V 8130 5300 50  0001 C CNN
 F 3 "~" H 8200 5300 50  0001 C CNN
 	1    8200 5300
@@
 F 0 "R16" H 8620 4796 50  0000 L CNN
 F 1 "R" H 8620 4705 50  0000 L CNN
-F 2 "Be-Elec:D_DO-35_SOD27_P10.16mm_Horizontal" V 8480 4750 50  0001 C CNN
+F 2 "Be-Elec:R_Axial_DIN0207_L6.3mm_D2.5mm_P10.16mm_Horizontal" V 8480 4750 50  0001 C CNN
 F 3 "~" H 8550 4750 50  0001 C CNN
 	1    8550 4750
@@
 F 0 "D2" H 8350 5266 50  0000 C CNN
 F 1 "1N4148" H 8350 5175 50  0000 C CNN
-F 2 "Diode_THT:D_DO-35_SOD27_P7.62mm_Horizontal" H 8350 4875 50  0001 C CNN
+F 2 "Be-Elec:D_DO-35_SOD27_P10.16mm_Horizontal" H 8350 4875 50  0001 C CNN
 F 3 "http://www.nxp.com/documents/data_sheet/1N4148_1N4448.pdf" H 8350 5050 50  0001 C CNN
 	1    8350 5050
@@
 F 0 "D1" V 7354 4529 50  0000 L CNN
 F 1 "1N4148" V 7445 4529 50  0000 L CNN
-F 2 "Diode_THT:D_DO-35_SOD27_P7.62mm_Horizontal" H 7400 4275 50  0001 C CNN
+F 2 "Be-Elec:D_DO-35_SOD27_P10.16mm_Horizontal" H 7400 4275 50  0001 C CNN
 F 3 "http://www.nxp.com/documents/data_sheet/1N4148_1N4448.pdf" H 7400 4450 50  0001 C CNN
 	1    7400 4450
@@
 F 0 "J2" H 9280 3942 50  0000 L CNN
 F 1 "Conn_01x02" H 9280 3851 50  0000 L CNN
-F 2 "Connector:JWT_A3963_1x02_P3.96mm_Vertical" H 9200 3950 50  0001 C CNN
+F 2 "Be-Elec:PhoenixContact_MSTBVA_2,5_2-G-5,08_1x02_P5.08mm_Vertical" H 9200 3950 50  0001 C CNN
 F 3 "~" H 9200 3950 50  0001 C CNN
 	1    9200 3950
@@
 F 0 "J3" H 820 6625 50  0000 C CNN
 F 1 "Conn_01x03" H 820 6716 50  0000 C CNN
-F 2 "Connector:FanPinHeader_1x03_P2.54mm_Vertical" H 900 6950 50  0001 C CNN
+F 2 "Be-Elec:PhoenixContact_MSTBVA_2,5_3-G-5,08_1x03_P5.08mm_Vertical" H 900 6950 50  0001 C CNN
 F 3 "~" H 900 6950 50  0001 C CNN
 	1    900  6950
@@
 	0    1    1    0
 $EndComp
-$Comp
-L BE_Amplificateur_Audio-cache:Relay:DIPxx-1Axx-12x U1
-U 1 1 5E77BED5
-P 8100 4150
-F 0 "U1" V 8567 4150 50  0000 C CNN
-F 1 "Relay_1CT" V 8476 4150 50  0000 C CNN
-F 2 "Relay_THT:Relay_StandexMeder_DIP_LowProfile" H 8450 4100 50  0001 L CNN
-F 3 "" H 8100 4150 50  0001 C CNN
-	1    8100 4150
-	0    -1   -1   0
-$EndComp
 Wire Wire Line
 	3650 3000 4050 3000
@@
 F 0 "Q4" H 4041 4596 50  0000 L CNN
 F 1 "2N2222" H 4041 4505 50  0000 L CNN
-F 2 "Package_TO_SOT_THT:TO-18-3" H 4050 4650 50  0001 C CNN
+F 2 "Be-Elec:TO-18-3" H 4050 4650 50  0001 C CNN
 F 3 "~" H 3850 4550 50  0001 C CNN
 	1    3850 4550
@@
 F 0 "Q5" H 4441 4946 50  0000 L CNN
 F 1 "2N2222" H 4441 4855 50  0000 L CNN
-F 2 "Package_TO_SOT_THT:TO-18-3" H 4450 5000 50  0001 C CNN
+F 2 "Be-Elec:TO-18-3" H 4450 5000 50  0001 C CNN
 F 3 "~" H 4250 4900 50  0001 C CNN
 	1    4250 4900
@@
 F 0 "Q8" H 4442 3646 50  0000 L CNN
 F 1 "BD139" H 4442 3555 50  0000 L CNN
-F 2 "Package_TO_SOT_THT:TO-126-3_Vertical" H 4450 3525 50  0001 L CIN
+F 2 "Be-Elec:TO-126-3_Vertical" H 4450 3525 50  0001 L CIN
 F 3 "http://www.st.com/internet/com/TECHNICAL_RESOURCES/TECHNICAL_LITERATURE/DATASHEET/CD00001225.pdf" H 4250 3600 50  0001 L CNN
 	1    4250 3600
@@
 F 0 "Q13" H 8041 5096 50  0000 L CNN
 F 1 "2N2222" H 8041 5005 50  0000 L CNN
-F 2 "Package_TO_SOT_THT:TO-18-3" H 8050 5150 50  0001 C CNN
+F 2 "Be-Elec:TO-18-3" H 8050 5150 50  0001 C CNN
 F 3 "~" H 7850 5050 50  0001 C CNN
 	1    7850 5050
@@
 F 0 "HS1" V 5603 3030 50  0000 L CNN
 F 1 "Heatsink" V 5694 3030 50  0000 L CNN
-F 2 "Heatsink:Heatsink_125x35x50mm_3xFixationM3" H 5662 2850 50  0001 C CNN
+F 2 "Be-Elec:Heatsink_Fischer_SK104-STC-STIC_35x13mm_2xDrill2.5mm" H 5662 2850 50  0001 C CNN
 F 3 "" H 5662 2850 50  0001 C CNN
 	1    5650 2850
@@
 F 0 "HS2" V 5603 5280 50  0000 L CNN
 F 1 "Heatsink" V 5694 5280 50  0000 L CNN
-F 2 "Heatsink:Heatsink_125x35x50mm_3xFixationM3" H 5662 5100 50  0001 C CNN
+F 2 "Be-Elec:Heatsink_Fischer_SK104-STC-STIC_35x13mm_2xDrill2.5mm" H 5662 5100 50  0001 C CNN
 F 3 "" H 5662 5100 50  0001 C CNN
 	1    5650 5100
@@
 Wire Wire Line
 	6650 4600 6650 4650
+$Comp
+L Relay:DIPxx-1Axx-12x U1
+U 1 1 5E76D2F3
+P 8100 4150
+F 0 "U1" V 8567 4150 50  0000 C CNN
+F 1 "Relay_1CT" V 8476 4150 50  0000 C CNN
+F 2 "Relay_THT:Relay_StandexMeder_DIP_LowProfile" H 8450 4100 50  0001 L CNN
+F 3 "https://standexelectronics.com/wp-content/uploads/datasheet_reed_relay_DIP.pdf" H 8100 4150 50  0001 C CNN
+	1    8100 4150
+	0    -1   -1   0
+$EndComp
 $EndSCHEMATC

Commit message: màj empreintes
manque à faire l'empreinte du relai
Parts:
- C1, C3, C4, C6: footprint Be-Elec:CP_Radial_D12.5mm_P5.00mm -> Be-Elec:CP_Radial_D8.0mm_P5.00mm
- C2: footprint Be-Elec:CP_Radial_D12.5mm_P5.00mm -> Be-Elec:C_Rect_L7.2mm_W3.5mm_P5.00mm_FKS2_FKP2_MKS2_MKP2
- Q10, Q12: footprint Be-Elec:TO-126-3_Vertical -> Be-Elec:TO-220-3_Vertical
- R11, R12: footprint Be-Elec:R_Axial_DIN0207_L6.3mm_D2.5mm_P10.16mm_Horizontal -> Be-Elec:R_Axial_DIN0516_L15.5mm_D5.0mm_P20.32mm_Horizontal
Changed lines of the file:
@@
 F 0 "C1" V 1145 4250 50  0000 C CNN
 F 1 "47µ" V 1236 4250 50  0000 C CNN
-F 2 "Be-Elec:CP_Radial_D12.5mm_P5.00mm" H 1438 4100 50  0001 C CNN
+F 2 "Be-Elec:CP_Radial_D8.0mm_P5.00mm" H 1438 4100 50  0001 C CNN
 F 3 "~" H 1400 4250 50  0001 C CNN
 	1    1400 4250
@@
 F 0 "C2" V 3448 4250 50  0000 C CNN
 F 1 "C" V 3539 4250 50  0000 C CNN
-F 2 "Be-Elec:CP_Radial_D12.5mm_P5.00mm" H 3738 4100 50  0001 C CNN
+F 2 "Be-Elec:C_Rect_L7.2mm_W3.5mm_P5.00mm_FKS2_FKP2_MKS2_MKP2" H 3738 4100 50  0001 C CNN
 F 3 "~" H 3700 4250 50  0001 C CNN
 	1    3700 4250
@@
 F 0 "R11" H 5620 3796 50  0000 L CNN
 F 1 "R" H 5620 3705 50  0000 L CNN
-F 2 "Be-Elec:R_Axial_DIN0207_L6.3mm_D2.5mm_P10.16mm_Horizontal" V 5480 3750 50  0001 C CNN
+F 2 "Be-Elec:R_Axial_DIN0516_L15.5mm_D5.0mm_P20.32mm_Horizontal" V 5480 3750 50  0001 C CNN
 F 3 "~" H 5550 3750 50  0001 C CNN
 	1    5550 3750
@@
 F 0 "R12" H 5620 4246 50  0000 L CNN
 F 1 "R" H 5620 4155 50  0000 L CNN
-F 2 "Be-Elec:R_Axial_DIN0207_L6.3mm_D2.5mm_P10.16mm_Horizontal" V 5480 4200 50  0001 C CNN
+F 2 "Be-Elec:R_Axial_DIN0516_L15.5mm_D5.0mm_P20.32mm_Horizontal" V 5480 4200 50  0001 C CNN
 F 3 "~" H 5550 4200 50  0001 C CNN
 	1    5550 4200
@@
 F 0 "C3" H 8668 5346 50  0000 L CNN
 F 1 "47µ" H 8668 5255 50  0000 L CNN
-F 2 "Be-Elec:CP_Radial_D12.5mm_P5.00mm" H 8588 5150 50  0001 C CNN
+F 2 "Be-Elec:CP_Radial_D8.0mm_P5.00mm" H 8588 5150 50  0001 C CNN
 F 3 "~" H 8550 5300 50  0001 C CNN
 	1    8550 5300
@@
 F 0 "C4" H 2218 6696 50  0000 L CNN
 F 1 "10µ" H 2218 6605 50  0000 L CNN
-F 2 "Be-Elec:CP_Radial_D12.5mm_P5.00mm" H 2138 6500 50  0001 C CNN
+F 2 "Be-Elec:CP_Radial_D8.0mm_P5.00mm" H 2138 6500 50  0001 C CNN
 F 3 "~" H 2100 6650 50  0001 C CNN
 	1    2100 6650
@@
 F 0 "C6" H 2218 7296 50  0000 L CNN
 F 1 "10µ" H 2218 7205 50  0000 L CNN
-F 2 "Be-Elec:CP_Radial_D12.5mm_P5.00mm" H 2138 7100 50  0001 C CNN
+F 2 "Be-Elec:CP_Radial_D8.0mm_P5.00mm" H 2138 7100 50  0001 C CNN
 F 3 "~" H 2100 7250 50  0001 C CNN
 	1    2100 7250
@@
 F 0 "Q12" H 5250 5250 50  0000 L CNN
 F 1 "TIP31" H 5250 5350 50  0000 L CNN
-F 2 "Be-Elec:TO-126-3_Vertical" H 5650 5200 50  0001 C CNN
+F 2 "Be-Elec:TO-220-3_Vertical" H 5650 5200 50  0001 C CNN
 F 3 "~" H 5450 5100 50  0001 C CNN
 	1    5450 5100
@@
 F 0 "Q10" H 5150 2650 50  0000 L CNN
 F 1 "TIP32" H 5150 2750 50  0000 L CNN
-F 2 "Be-Elec:TO-126-3_Vertical" H 5650 2950 50  0001 C CNN
+F 2 "Be-Elec:TO-220-3_Vertical" H 5650 2950 50  0001 C CNN
 F 3 "~" H 5450 2850 50  0001 C CNN
 	1    5450 2850

Commit message: empreinte du relai: ok
Parts:
- U1: footprint Relay_THT:Relay_StandexMeder_DIP_LowProfile -> Be-Elec:RelayBE
Changed lines of the file:
@@
 F 0 "U1" V 8567 4150 50  0000 C CNN
 F 1 "Relay_1CT" V 8476 4150 50  0000 C CNN
-F 2 "Relay_THT:Relay_StandexMeder_DIP_LowProfile" H 8450 4100 50  0001 L CNN
+F 2 "Be-Elec:RelayBE" H 8450 4100 50  0001 L CNN
 F 3 "https://standexelectronics.com/wp-content/uploads/datasheet_reed_relay_DIP.pdf" H 8100 4150 50  0001 C CNN
 	1    8100 4150
