File: BE_Amplificateur_Audio/BE_Amplificateur_Audio.sch (KiCad schematic (older format))
At the start: 52 parts, among them J2 Conn_01x02, J3 Conn_01x03, Q1 2N2907, Q10 TIP32, Q11 BD138, Q12 TIP31, Q13 2N2222, Q2 2N2907, Q3 2N2907, Q4 2N2222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

Commit message: Modifs après avis
Modifications après 1er avis de placement et routage
Parts:
- removed Q12: TIP31, Be-Elec:TO-220-3_Vertical, symbol Device:Q_PNP_BCE
- added Q12: TIP31, Be-Elec:TO-220-3_Vertical, symbol Device:Q_NPN_BCE
Changed lines of the file:
@@
-$EndComp
-$Comp
-L Device:Q_PNP_BCE Q12
-U 1 1 5E7A59B1
-P 5450 5100
-F 0 "Q12" H 5250 5250 50  0000 L CNN
-F 1 "TIP31" H 5250 5350 50  0000 L CNN
-F 2 "Be-Elec:TO-220-3_Vertical" H 5650 5200 50  0001 C CNN
-F 3 "~" H 5450 5100 50  0001 C CNN
-	1    5450 5100
-	1    0    0    1
 $EndComp
 $Comp
@@
 	1    0    0    -1
 $EndComp
+$Comp
+L Device:Q_NPN_BCE Q12
+U 1 1 5EA2271D
+P 5450 5100
+F 0 "Q12" H 5641 5146 50  0000 L CNN
+F 1 "TIP31" H 5641 5055 50  0000 L CNN
+F 2 "Be-Elec:TO-220-3_Vertical" H 5650 5200 50  0001 C CNN
+F 3 "~" H 5450 5100 50  0001 C CNN
+	1    5450 5100
+	1    0    0    -1
+$EndComp

Commit message: Corrections au niveau de Q7
J'ai corrigé les PWRFLAG et trouvé une erreur au niveau de Q7 : il manquait un fil. C'est corrigé et le routage est mis à jour.
Connections:
- wire segments 147 -> 155
- no-connect marks 0 -> 3
Changed lines of the file:
@@
 	3000 3950 3000 4050
-Wire Wire Line
-	3000 4450 3000 4650
 Wire Wire Line
 	2200 4950 2200 5000
@@
 L Device:R R10
 U 1 1 5E696E1E
-P 3350 3350
-F 0 "R10" H 3420 3396 50  0000 L CNN
-F 1 "R" H 3420 3305 50  0000 L CNN
-F 2 "Be-Elec:R_Axial_DIN0207_L6.3mm_D2.5mm_P10.16mm_Horizontal" V 3280 3350 50  0001 C CNN
-F 3 "~" H 3350 3350 50  0001 C CNN
-	1    3350 3350
+P 3350 3450
+F 0 "R10" H 3420 3496 50  0000 L CNN
+F 1 "R" H 3420 3405 50  0000 L CNN
+F 2 "Be-Elec:R_Axial_DIN0207_L6.3mm_D2.5mm_P10.16mm_Horizontal" V 3280 3450 50  0001 C CNN
+F 3 "~" H 3350 3450 50  0001 C CNN
+	1    3350 3450
 	1    0    0    -1
 $EndComp
@@
 L Device:R_POT RV2
 U 1 1 5E697543
-P 3350 3700
-F 0 "RV2" H 3280 3746 50  0000 R CNN
-F 1 "R_POT" H 3280 3655 50  0000 R CNN
-F 2 "Be-Elec:Potentiometer_Bourns_3296W_Vertical" H 3350 3700 50  0001 C CNN
-F 3 "~" H 3350 3700 50  0001 C CNN
-	1    3350 3700
-	1    0    0    -1
-$EndComp
-Wire Wire Line
-	3350 3500 3350 3550
-Wire Wire Line
-	3500 3700 3500 3500
-Wire Wire Line
-	3500 3500 3350 3500
-Connection ~ 3350 3500
+P 3350 3800
+F 0 "RV2" H 3280 3846 50  0000 R CNN
+F 1 "R_POT" H 3280 3755 50  0000 R CNN
+F 2 "Be-Elec:Potentiometer_Bourns_3296W_Vertical" H 3350 3800 50  0001 C CNN
+F 3 "~" H 3350 3800 50  0001 C CNN
+	1    3350 3800
+	1    0    0    -1
+$EndComp
+Wire Wire Line
+	3350 3600 3350 3650
+Wire Wire Line
+	3500 3800 3500 3600
+Wire Wire Line
+	3500 3600 3350 3600
+Connection ~ 3350 3600
 $Comp
 L power:GND #PWR0105
 U 1 1 5E697B7E
-P 3350 3850
-F 0 "#PWR0105" H 3350 3600 50  0001 C CNN
-F 1 "GND" H 3355 3677 50  0000 C CNN
-F 2 "" H 3350 3850 50  0001 C CNN
-F 3 "" H 3350 3850 50  0001 C CNN
-	1    3350 3850
+P 3350 3950
+F 0 "#PWR0105" H 3350 3700 50  0001 C CNN
+F 1 "GND" H 3355 3777 50  0000 C CNN
+F 2 "" H 3350 3950 50  0001 C CNN
+F 3 "" H 3350 3950 50  0001 C CNN
+	1    3350 3950
 	1    0    0    -1
 $EndComp
@@
 $EndComp
 Wire Wire Line
-	3650 3000 4050 3000
+	3650 3000 3700 3000
 Wire Wire Line
 	6500 4600 6500 4800
@@
 	1    0    0    -1
 $EndComp
+$Comp
+L power:PWR_FLAG #FLG0101
+U 1 1 5EA2FD8C
+P 4500 6500
+F 0 "#FLG0101" H 4500 6575 50  0001 C CNN
+F 1 "PWR_FLAG" H 4500 6674 50  0000 C CNN
+F 2 "" H 4500 6500 50  0001 C CNN
+F 3 "~" H 4500 6500 50  0001 C CNN
+	1    4500 6500
+	1    0    0    -1
+$EndComp
+$Comp
+L power:PWR_FLAG #FLG0102
+U 1 1 5EA301E2
+P 4900 6500
+F 0 "#FLG0102" H 4900 6575 50  0001 C CNN
+F 1 "PWR_FLAG" H 4900 6674 50  0000 C CNN
+F 2 "" H 4900 6500 50  0001 C CNN
+F 3 "~" H 4900 6500 50  0001 C CNN
+	1    4900 6500
+	1    0    0    -1
+$EndComp
+$Comp
+L power:PWR_FLAG #FLG0103
+U 1 1 5EA30255
+P 4100 6850
+F 0 "#FLG0103" H 4100 6925 50  0001 C CNN
+F 1 "PWR_FLAG" H 4100 7023 50  0000 C CNN
+F 2 "" H 4100 6850 50  0001 C CNN
+F 3 "~" H 4100 6850 50  0001 C CNN
+	1    4100 6850
+	-1   0    0    1
+$EndComp
+$Comp
+L power:GND #PWR0119
+U 1 1 5EA30330
+P 4500 6850
+F 0 "#PWR0119" H 4500 6600 50  0001 C CNN
+F 1 "GND" H 4505 6677 50  0000 C CNN
+F 2 "" H 4500 6850 50  0001 C CNN
+F 3 "" H 4500 6850 50  0001 C CNN
+	1    4500 6850
+	1    0    0    -1
+$EndComp
+$Comp
+L power:-12V #PWR0120
+U 1 1 5EA303A3
+P 4900 6850
+F 0 "#PWR0120" H 4900 6950 50  0001 C CNN
+F 1 "-12V" H 4915 7023 50  0000 C CNN
+F 2 "" H 4900 6850 50  0001 C CNN
+F 3 "" H 4900 6850 50  0001 C CNN
+	1    4900 6850
+	-1   0    0    1
+$EndComp
+$Comp
+L power:+12V #PWR0121
+U 1 1 5EA30416
+P 4100 6500
+F 0 "#PWR0121" H 4100 6350 50  0001 C CNN
+F 1 "+12V" H 4115 6673 50  0000 C CNN
+F 2 "" H 4100 6500 50  0001 C CNN
+F 3 "" H 4100 6500 50  0001 C CNN
+	1    4100 6500
+	1    0    0    -1
+$EndComp
+Wire Wire Line
+	4100 6500 4100 6850
+Wire Wire Line
+	4500 6500 4500 6850
+Wire Wire Line
+	4900 6500 4900 6850
+NoConn ~ 1250 4150
+NoConn ~ 5550 2200
+NoConn ~ 5200 1650
+Wire Wire Line
+	3000 4450 3000 4650
+Wire Wire Line
+	3350 3300 3350 3250
+Wire Wire Line
+	3350 3250 3700 3250
+Wire Wire Line
+	3700 3250 3700 3000
+Connection ~ 3350 3250
+Wire Wire Line
+	3350 3250 3350 3200
+Connection ~ 3700 3000
+Wire Wire Line
+	3700 3000 4050 3000
 $EndSCHEMATC
