File: BE_Amplificateur_Audio/BE_Amplificateur_Audio_v0.kicad_pcb (KiCad board)
At the start: 2 copper layers, 110 x 100 mm, 52 parts, among them J2 Conn_01x02, J3 Conn_01x03, Q1 2N2907, Q10 TIP32, Q11 BD138, Q12 TIP31, Q13 2N2222, Q2 2N2907, Q3 2N2907, Q4 2N2222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

Commit message: Placement + Routage
Placement + routage (v0 à v2)
Parts:
- moved U2 71.1 mm to (68.2, 121.8), turned to 90 degrees
Routing:
- net Net-(C1-Pad2): track 76.2 -> 12.3 mm
- net GND: track 0.00 -> 31.7 mm
- net Net-(C3-Pad1): track 0.04 -> 12.8 mm
- net -12V: track 246.0 -> 256.3 mm
- net Net-(D1-Pad2): track 69.6 -> 70.3 mm
- removed copper zone on B.Cu, net +12V
- removed copper zone on B.Cu, net -12V
- removed copper zone on B.Cu, net Net-(C2-Pad1)
- removed copper zone on B.Cu, net Net-(C3-Pad1)
- removed copper zone on B.Cu, net Net-(R10-Pad2)
