File: BE_Amplificateur_Audio/Jack_bas/BE_Amplificateur_Audio_jack_bas.kicad_pcb (KiCad board)
At the start: 2 copper layers, 110 x 100 mm, 52 parts, among them J2 Conn_01x02, J3 Conn_01x03, Q1 2N2907, Q10 TIP32, Q11 BD138, Q12 TIP31, Q13 2N2222, Q2 2N2907, Q3 2N2907, Q4 2N2222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

Commit message: PRET POUR VERIF
Problème de librairie de symboles qui est apparu --> résolu
Schematic à jour.
Netliste à jour.
Placement à jour.
Routage à jour.
Prêt pour vérification du placement et routage.
Parts:
- moved U2 72.5 mm to (66.8, 121.4), turned to 90 degrees
Routing:
- net Net-(C1-Pad2): track 76.2 -> 10.4 mm
Changed lines of the file:
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@@
     (thickness 1.6)
     (drawings 6)
-    (tracks 250)
+    (tracks 248)
     (zones 0)
     (modules 52)
@@
   )
   (module Be-Elec:Jack_35RAPC2AV (layer F.Cu)
-    (at 136.8679 103.0859 180)
-    (fp_text reference U2 (at 1.1 6.7 180) (layer F.SilkS)
+    (at 66.76644 121.39168 90)
+    (fp_text reference U2 (at 1.1 6.7 90) (layer F.SilkS)
       (effects (font (size 1 1) (thickness 0.15)))
     )
-    (fp_text value Jack_Mono (at -0.8 -5.6 180) (layer F.Fab)
+    (fp_text value Jack_Mono (at -0.8 -5.6 90) (layer F.Fab)
       (effects (font (size 1 1) (thickness 0.15)))
     )
@@
     (fp_line (start 0 -3) (end -4 -3) (layer F.SilkS) (width 0.15))
     (fp_line (start 0 -3) (end 0 3) (layer F.SilkS) (width 0.15))
-    (fp_text user %R (at -4.3 6.6 180) (layer F.Fab)
+    (fp_text user %R (at -4.3 6.6 90) (layer F.Fab)
       (effects (font (size 1 1) (thickness 0.15)))
     )
-    (pad TN thru_hole circle (at 13.2 0 180) (size 3.5 3.5) (drill 2) (layers *.Cu *.Mask)
+    (pad TN thru_hole circle (at 13.2 0 90) (size 3.5 3.5) (drill 2) (layers *.Cu *.Mask)
       (net 32 "Net-(U2-PadTN)"))
-    (pad G thru_hole circle (at 2.1 0 180) (size 3.5 3.5) (drill 2) (layers *.Cu *.Mask)
+    (pad G thru_hole circle (at 2.1 0 90) (size 3.5 3.5) (drill 2) (layers *.Cu *.Mask)
       (net 7 GND))
-    (pad T thru_hole circle (at 7.4 0 180) (size 3.5 3.5) (drill 2) (layers *.Cu *.Mask)
+    (pad T thru_hole circle (at 7.4 0 90) (size 3.5 3.5) (drill 2) (layers *.Cu *.Mask)
       (net 2 "Net-(C1-Pad2)"))
   )
@@
   (segment (start 49.1998 103.6066) (end 41.9608 96.3676) (width 1.5) (layer B.Cu) (net 1))
   (segment (start 54.1655 103.6066) (end 49.1998 103.6066) (width 1.5) (layer B.Cu) (net 1))
-  (segment (start 61.3499 105.791) (end 67.8015 112.2426) (width 1.5) (layer B.Cu) (net 2))
-  (segment (start 129.4679 105.7996) (end 129.4679 103.0859) (width 1.5) (layer B.Cu) (net 2))
-  (segment (start 123.0249 112.2426) (end 129.4679 105.7996) (width 1.5) (layer B.Cu) (net 2))
-  (segment (start 67.8015 112.2426) (end 123.0249 112.2426) (width 1.5) (layer B.Cu) (net 2))
+  (segment (start 61.3499 108.57514) (end 66.76644 113.99168) (width 1.5) (layer B.Cu) (net 2))
+  (segment (start 61.3499 105.791) (end 61.3499 108.57514) (width 1.5) (layer B.Cu) (net 2))
   (segment (start 61.9252 61.8363) (end 64.4525 64.3636) (width 1.5) (layer B.Cu) (net 3))
   (segment (start 52.2986 61.8363) (end 61.9252 61.8363) (width 1.5) (layer B.Cu) (net 3))
